Commit message: Stabilize three-arm demo startup and execution flow

File: catkin_ws/src/my_arm_description/urdf/three_arms_new.urdf (robot description, URDF)
Before this commit: robot three_4dof_arms, 41 links, 40 joints
Joints:
- joint arm1_J1: limit lower=0 upper=6.28 effort=0.17658 velocity=8.727 -> lower=0 upper=6.28 effort=0.5 velocity=8.727
- joint arm1_J2: limit lower=-1.57 upper=1.57 effort=0.17658 velocity=8.727 -> lower=-1.57 upper=1.57 effort=0.5 velocity=8.727
- joint arm1_J3: limit lower=-1.57 upper=1.57 effort=0.17658 velocity=8.727 -> lower=-1.57 upper=1.57 effort=0.5 velocity=8.727
- joint arm1_J4: limit lower=-1.57 upper=1.57 effort=0.17658 velocity=8.727 -> lower=-1.57 upper=1.57 effort=0.5 velocity=8.727
- joint arm1_J5: limit lower=-1.57 upper=1.57 effort=0.17658 velocity=8.727 -> lower=-1.57 upper=1.57 effort=0.5 velocity=8.727
- joint arm1_J611: limit lower=-1.57 upper=0 effort=0.17658 velocity=8.727 -> lower=-1.57 upper=0 effort=0.5 velocity=8.727
- joint arm1_J612: limit lower=0 upper=3.14 effort=0.17658 velocity=8.727 -> lower=0 upper=3.14 effort=0.5 velocity=8.727
- joint arm1_J613: limit lower=0 upper=3.14 effort=0.17658 velocity=8.727 -> lower=0 upper=3.14 effort=0.5 velocity=8.727
- joint arm1_J621: limit lower=-1.57 upper=0 effort=0.17658 velocity=8.727 -> lower=-1.57 upper=0 effort=0.5 velocity=8.727
- joint arm1_J622: limit lower=0 upper=3.14 effort=0.17658 velocity=8.727 -> lower=0 upper=3.14 effort=0.5 velocity=8.727
- joint arm1_J623: limit lower=0 upper=3.14 effort=0.17658 velocity=8.727 -> lower=0 upper=3.14 effort=0.5 velocity=8.727
- joint arm2_J1: limit lower=0 upper=6.28 effort=0.17658 velocity=8.727 -> lower=0 upper=6.28 effort=0.5 velocity=8.727
- joint arm2_J2: limit lower=-1.57 upper=1.57 effort=0.17658 velocity=8.727 -> lower=-1.57 upper=1.57 effort=0.5 velocity=8.727
- joint arm2_J3: limit lower=-1.57 upper=1.57 effort=0.17658 velocity=8.727 -> lower=-1.57 upper=1.57 effort=0.5 velocity=8.727
- joint arm2_J4: limit lower=-1.57 upper=1.57 effort=0.17658 velocity=8.727 -> lower=-1.57 upper=1.57 effort=0.5 velocity=8.727
- joint arm2_J5: limit lower=-1.57 upper=1.57 effort=0.17658 velocity=8.727 -> lower=-1.57 upper=1.57 effort=0.5 velocity=8.727
- joint arm2_J611: limit lower=-1.57 upper=0 effort=0.17658 velocity=8.727 -> lower=-1.57 upper=0 effort=0.5 velocity=8.727
- joint arm2_J612: limit lower=0 upper=3.14 effort=0.17658 velocity=8.727 -> lower=0 upper=3.14 effort=0.5 velocity=8.727
- joint arm2_J613: limit lower=0 upper=3.14 effort=0.17658 velocity=8.727 -> lower=0 upper=3.14 effort=0.5 velocity=8.727
- joint arm2_J621: limit lower=-1.57 upper=0 effort=0.17658 velocity=8.727 -> lower=-1.57 upper=0 effort=0.5 velocity=8.727
- joint arm2_J622: limit lower=0 upper=3.14 effort=0.17658 velocity=8.727 -> lower=0 upper=3.14 effort=0.5 velocity=8.727
- joint arm2_J623: limit lower=0 upper=3.14 effort=0.17658 velocity=8.727 -> lower=0 upper=3.14 effort=0.5 velocity=8.727

File: catkin_ws/src/my_three_arms_moveit_config/config/gazebo_three_4dof_arms.urdf (robot description, URDF)
Before this commit: robot three_4dof_arms, 38 links, 37 joints
Links:
- added link arm1_tcp
- added link arm2_tcp
- added link arm3_tcp
Joints:
- added joint arm1_tcp_joint: type fixed, parent arm1_J5_Link, child arm1_tcp, origin xyz=0.065485 0.0064933 -0.0162493 rpy=0 0 0
- added joint arm2_tcp_joint: type fixed, parent arm2_J5_Link, child arm2_tcp, origin xyz=0.065485 0.0064933 -0.0162493 rpy=0 0 0
- added joint arm3_tcp_joint: type fixed, parent arm3_J5_Link, child arm3_tcp, origin xyz=0.065485 0.0064933 -0.0162493 rpy=0 0 0
- joint arm1_J1: limit lower=0 upper=6.28 effort=0.17658 velocity=8.727 -> lower=0 upper=6.28 effort=1.0 velocity=8.727
- joint arm1_J2: limit lower=-1.57 upper=1.57 effort=0.17658 velocity=8.727 -> lower=-1.57 upper=1.57 effort=1.0 velocity=8.727
- joint arm1_J3: limit lower=-1.57 upper=1.57 effort=0.17658 velocity=8.727 -> lower=-1.57 upper=1.57 effort=1.0 velocity=8.727
- joint arm1_J4: limit lower=-1.57 upper=1.57 effort=0.17658 velocity=8.727 -> lower=-1.57 upper=1.57 effort=1.0 velocity=8.727
- joint arm1_J5: limit lower=-1.57 upper=1.57 effort=0.17658 velocity=8.727 -> lower=-1.57 upper=1.57 effort=1.0 velocity=8.727
- joint arm1_J611: limit lower=-1.57 upper=0 effort=0.17658 velocity=8.727 -> lower=-1.57 upper=0 effort=1.0 velocity=8.727
- joint arm1_J612: limit lower=0 upper=3.14 effort=0.17658 velocity=8.727 -> lower=0 upper=3.14 effort=1.0 velocity=8.727
- joint arm1_J613: limit lower=0 upper=3.14 effort=0.17658 velocity=8.727 -> lower=0 upper=3.14 effort=1.0 velocity=8.727
- joint arm1_J621: limit lower=-1.57 upper=0 effort=0.17658 velocity=8.727 -> lower=-1.57 upper=0 effort=1.0 velocity=8.727
- joint arm1_J622: limit lower=0 upper=3.14 effort=0.17658 velocity=8.727 -> lower=0 upper=3.14 effort=1.0 velocity=8.727
- joint arm1_J623: limit lower=0 upper=3.14 effort=0.17658 velocity=8.727 -> lower=0 upper=3.14 effort=1.0 velocity=8.727
- joint arm2_J1: limit lower=0 upper=6.28 effort=0.17658 velocity=8.727 -> lower=0 upper=6.28 effort=1.0 velocity=8.727
- joint arm2_J2: limit lower=-1.57 upper=1.57 effort=0.17658 velocity=8.727 -> lower=-1.57 upper=1.57 effort=1.0 velocity=8.727
- joint arm2_J3: limit lower=-1.57 upper=1.57 effort=0.17658 velocity=8.727 -> lower=-1.57 upper=1.57 effort=1.0 velocity=8.727
- joint arm2_J4: limit lower=-1.57 upper=1.57 effort=0.17658 velocity=8.727 -> lower=-1.57 upper=1.57 effort=1.0 velocity=8.727
- joint arm2_J5: limit lower=-1.57 upper=1.57 effort=0.17658 velocity=8.727 -> lower=-1.57 upper=1.57 effort=1.0 velocity=8.727
- joint arm2_J611: limit lower=-1.57 upper=0 effort=0.17658 velocity=8.727 -> lower=-1.57 upper=0 effort=1.0 velocity=8.727
- joint arm2_J612: limit lower=0 upper=3.14 effort=0.17658 velocity=8.727 -> lower=0 upper=3.14 effort=1.0 velocity=8.727
- joint arm2_J613: limit lower=0 upper=3.14 effort=0.17658 velocity=8.727 -> lower=0 upper=3.14 effort=1.0 velocity=8.727
- joint arm2_J621: limit lower=-1.57 upper=0 effort=0.17658 velocity=8.727 -> lower=-1.57 upper=0 effort=1.0 velocity=8.727
- joint arm2_J622: limit lower=0 upper=3.14 effort=0.17658 velocity=8.727 -> lower=0 upper=3.14 effort=1.0 velocity=8.727
- joint arm2_J623: limit lower=0 upper=3.14 effort=0.17658 velocity=8.727 -> lower=0 upper=3.14 effort=1.0 velocity=8.727
- joint arm3_J1: limit lower=0 upper=6.28 effort=0.17658 velocity=8.727 -> lower=0 upper=6.28 effort=1.0 velocity=8.727
- joint arm3_J2: limit lower=-1.57 upper=1.57 effort=0.17658 velocity=8.727 -> lower=-1.57 upper=1.57 effort=1.0 velocity=8.727
- joint arm3_J3: limit lower=-1.57 upper=1.57 effort=0.17658 velocity=8.727 -> lower=-1.57 upper=1.57 effort=1.0 velocity=8.727
- joint arm3_J4: limit lower=-1.57 upper=1.57 effort=0.17658 velocity=8.727 -> lower=-1.57 upper=1.57 effort=1.0 velocity=8.727
- joint arm3_J5: limit lower=-1.57 upper=1.57 effort=0.17658 velocity=8.727 -> lower=-1.57 upper=1.57 effort=1.0 velocity=8.727
- joint arm3_J611: limit lower=-1.57 upper=0 effort=0.17658 velocity=8.727 -> lower=-1.57 upper=0 effort=1.0 velocity=8.727
- joint arm3_J612: limit lower=0 upper=3.14 effort=0.17658 velocity=8.727 -> lower=0 upper=3.14 effort=1.0 velocity=8.727
- joint arm3_J613: limit lower=0 upper=3.14 effort=0.17658 velocity=8.727 -> lower=0 upper=3.14 effort=1.0 velocity=8.727
- joint arm3_J621: limit lower=-1.57 upper=0 effort=0.17658 velocity=8.727 -> lower=-1.57 upper=0 effort=1.0 velocity=8.727
- joint arm3_J622: limit lower=0 upper=3.14 effort=0.17658 velocity=8.727 -> lower=0 upper=3.14 effort=1.0 velocity=8.727
- joint arm3_J623: limit lower=0 upper=3.14 effort=0.17658 velocity=8.727 -> lower=0 upper=3.14 effort=1.0 velocity=8.727
